Commit message: feat(g1_tt): integrate real-mesh paddle + fix body/event remaps + FK-calibrate geometry
- Adopt user's regenerated real-mesh paddle (tt_paddle.stl, base rev_1_0,
  merged right_tt_paddle_link, contact @ wrist +X 0.337m). paddle_offset 0.302->0.337.
- Fix fixed-joint-merge name resolution: paddel_head_too_near head_link->torso_link;
  remap reset_locomotion_joints / reset_manipulation_joints to G1 joint names.
- Stance: wbt-proven leg bend (hip -0.312/knee 0.669/ankle -0.363); robot stands
  stably at pelvis z~0.685 (verified via probe, 200 steps steady).
- FK calibration: hit_body_height 0.685, paddle_y_offset -0.227.
- Probe: add z-trajectory + result-file output (Kit clobbers stdout).

Co-Authored-By: Claude Opus 4.8 <noreply@anthropic.com>

File: legged_lab/assets/unitree/g1_description/g1_23dof_tt.urdf (robot description, URDF)
Before this commit: robot g1_23dof, 33 links, 32 joints
Links:
- removed link waist_support_link
- removed link waist_yaw_fixed_link
- link torso_link: mass 8.562 -> 6.78; geometry collision mesh filename=meshes/torso_link_23dof_rev_1_0.STL; visual mesh filename=meshes/torso_link_23dof_rev_1_0.STL
Joints:
- removed joint waist_support_joint
- removed joint waist_yaw_fixed_joint
- joint d435_joint: origin xyz=0.0576235 0.01753 0.41987 rpy=0 0.8307767239493009 0 -> xyz=0.0576235 0.01753 0.42987 rpy=0 0.8307767239493009 0
- joint head_joint: origin xyz=0.0039635 0 -0.054 rpy=0 0 0 -> xyz=0.0039635 0 -0.044 rpy=0 0 0
- joint imu_in_torso_joint: origin xyz=-0.03959 -0.00224 0.13792 rpy=0 0 0 -> xyz=-0.03959 -0.00224 0.14792 rpy=0 0 0
- joint left_hip_roll_joint: limit lower=-0.5236 upper=2.9671 effort=88 velocity=32 -> lower=-0.5236 upper=2.9671 effort=139 velocity=20
- joint left_shoulder_pitch_joint: origin xyz=0.0039563 0.10022 0.23778 rpy=0.27931 5.4949E-05 -0.00019159 -> xyz=0.0039563 0.10022 0.24778 rpy=0.27931 5.4949E-05 -0.00019159
- joint logo_joint: origin xyz=0.0039635 0 -0.054 rpy=0 0 0 -> xyz=0.0039635 0 -0.044 rpy=0 0 0
- joint mid360_joint: origin xyz=0.0002835 0.00003 0.40618 rpy=0 0.04014257279586953 0 -> xyz=0.0002835 0.00003 0.41618 rpy=0 0.04014257279586953 0
- joint right_hip_roll_joint: limit lower=-2.9671 upper=0.5236 effort=88 velocity=32 -> lower=-2.9671 upper=0.5236 effort=139 velocity=20
- joint right_shoulder_pitch_joint: origin xyz=0.0039563 -0.10021 0.23778 rpy=-0.27931 5.4949E-05 0.00019159 -> xyz=0.0039563 -0.10021 0.24778 rpy=-0.27931 5.4949E-05 0.00019159
- joint waist_yaw_joint: origin xyz=-0.0039635 0 0.054 rpy=0 0 0 -> xyz=-0.0039635 0 0.044 rpy=0 0 0

File: legged_lab/assets/unitree/g1_description/g1_23dof_tt_paddle.urdf (robot description, URDF)
Before this commit: robot g1_23dof, 41 links, 40 joints
Links:
- removed link right_tt_paddle_blade_link
- removed link right_tt_paddle_handle_link
- removed link waist_support_link
- removed link waist_yaw_fixed_link
- added link right_tt_paddle_link, mass 0.17; collision box size=0.075 0.032 0.022; collision cylinder length=0.005 radius=0.075
- link right_tt_paddle_holder_link: geometry collision box size=0.075 0.04 0.026; visual box size=0.075 0.004 0.022
- link torso_link: mass 8.562 -> 6.78; geometry collision mesh filename=meshes/torso_link_23dof_rev_1_0.STL; visual mesh filename=meshes/torso_link_23dof_rev_1_0.STL
Joints:
- removed joint right_tt_paddle_blade_joint
- removed joint right_tt_paddle_handle_joint
- removed joint waist_support_joint
- removed joint waist_yaw_fixed_joint
- added joint right_tt_paddle_joint: type fixed, parent right_tt_paddle_holder_link, child right_tt_paddle_link, origin xyz=0.0 0 0 rpy=0 0 0
- joint d435_joint: origin xyz=0.0576235 0.01753 0.41987 rpy=0 0.8307767239493009 0 -> xyz=0.0576235 0.01753 0.42987 rpy=0 0.8307767239493009 0
- joint head_joint: origin xyz=0.0039635 0 -0.054 rpy=0 0 0 -> xyz=0.0039635 0 -0.044 rpy=0 0 0
- joint imu_in_torso_joint: origin xyz=-0.03959 -0.00224 0.13792 rpy=0 0 0 -> xyz=-0.03959 -0.00224 0.14792 rpy=0 0 0
- joint left_hip_roll_joint: limit lower=-0.5236 upper=2.9671 effort=88 velocity=32 -> lower=-0.5236 upper=2.9671 effort=139 velocity=20
- joint left_shoulder_pitch_joint: origin xyz=0.0039563 0.10022 0.23778 rpy=0.27931 5.4949E-05 -0.00019159 -> xyz=0.0039563 0.10022 0.24778 rpy=0.27931 5.4949E-05 -0.00019159
- joint logo_joint: origin xyz=0.0039635 0 -0.054 rpy=0 0 0 -> xyz=0.0039635 0 -0.044 rpy=0 0 0
- joint mid360_joint: origin xyz=0.0002835 0.00003 0.40618 rpy=0 0.04014257279586953 0 -> xyz=0.0002835 0.00003 0.41618 rpy=0 0.04014257279586953 0
- joint right_hip_roll_joint: limit lower=-2.9671 upper=0.5236 effort=88 velocity=32 -> lower=-2.9671 upper=0.5236 effort=139 velocity=20
- joint right_paddle_contact_frame_joint: origin xyz=0 0 0.003 rpy=0 0 0 -> xyz=0.165 0 0.0025 rpy=0 0 0; parent right_tt_paddle_blade_link -> right_tt_paddle_link
- joint right_shoulder_pitch_joint: origin xyz=0.0039563 -0.10021 0.23778 rpy=-0.27931 5.4949E-05 0.00019159 -> xyz=0.0039563 -0.10021 0.24778 rpy=-0.27931 5.4949E-05 0.00019159
- joint waist_yaw_joint: origin xyz=-0.0039635 0 0.054 rpy=0 0 0 -> xyz=-0.0039635 0 0.044 rpy=0 0 0
