Commit message: feat(assets): adopt PACE paddle adapter (g1_23dof_tt_paddle.urdf), replace placeholder
- Vendor user's PACE-style fixed paddle fixture (xacro + stdlib generator + base
  g1_23dof.urdf + ready-to-load g1_23dof_tt_paddle.urdf, 23 DoF preserved, blade
  has collision). Overwrites the placeholder primitive paddle URDF from Task 2.
- G1_TT_CFG asset_path -> g1_23dof_tt_paddle.urdf.
- paddle_offset -> (0.302,0,0): contact point along wrist +X (mount+ext+blade);
  paddle_body_name stays right_wrist_roll_rubber_hand (rigid offset, robust to
  fixed-joint merge; blade collision still rebounds the ball). FK-calibrated later.

Co-Authored-By: Claude Opus 4.8 <noreply@anthropic.com>

File: legged_lab/assets/unitree/g1_description/g1_23dof_tt_paddle.urdf (robot description, URDF)
Before this commit: robot g1_23dof, 33 links, 32 joints
Links:
- added link right_adapter_mount_frame, mass 1e-6
- added link right_paddle_contact_frame, mass 1e-6
- added link right_paddle_handle_frame, mass 1e-6
- added link right_tt_adapter_mount_link, mass 0.03; collision cylinder length=0.012 radius=0.025; visual cylinder length=0.012 radius=0.025
- added link right_tt_extension_link, mass 0.08; collision cylinder length=0.16 radius=0.018; visual cylinder length=0.16 radius=0.018
- added link right_tt_paddle_blade_link, mass 0.13; collision cylinder length=0.006 radius=0.075; visual cylinder length=0.006 radius=0.075
- added link right_tt_paddle_handle_link, mass 0.04; collision box size=0.095 0.028 0.013; visual box size=0.095 0.028 0.013
- added link right_tt_paddle_holder_link, mass 0.05; collision box size=0.075 0.038 0.02; visual box size=0.075 0.004 0.016
Joints:
- added joint right_adapter_mount_frame_joint: type fixed, parent right_tt_adapter_mount_link, child right_adapter_mount_frame, origin xyz=0 0 0 rpy=0 0 0
- added joint right_paddle_contact_frame_joint: type fixed, parent right_tt_paddle_blade_link, child right_paddle_contact_frame, origin xyz=0 0 0.003 rpy=0 0 0
- added joint right_paddle_handle_frame_joint: type fixed, parent right_tt_paddle_holder_link, child right_paddle_handle_frame, origin xyz=0.0375 0 0 rpy=0 0 0
- added joint right_tt_adapter_mount_joint: type fixed, parent right_wrist_roll_rubber_hand, child right_tt_adapter_mount_link, origin xyz=0 0 0 rpy=0 0 0
- added joint right_tt_extension_joint: type fixed, parent right_tt_adapter_mount_link, child right_tt_extension_link, origin xyz=0.012 0 0 rpy=0 0 0
- added joint right_tt_paddle_blade_joint: type fixed, parent right_tt_paddle_handle_link, child right_tt_paddle_blade_link, origin xyz=0.13 0 0 rpy=0 0 0
- added joint right_tt_paddle_handle_joint: type fixed, parent right_tt_paddle_holder_link, child right_tt_paddle_handle_link, origin xyz=0.0 0 0 rpy=0 0 0
- added joint right_tt_paddle_holder_joint: type fixed, parent right_tt_extension_link, child right_tt_paddle_holder_link, origin xyz=0.16 0 0 rpy=0 0 0

Commit message: fix(g1_tt): roll paddle holder +90deg about +X so blade face is lateral/forward
Diagnosis (contact_probe): trained policy hit 84% but ball went backward
(vx=-5.4), blade face pointed UP (+Z normal) at contact -> ball never cleared
the net (pass_net~0, success~0). Root cause = paddle face normal perpendicular
to forearm + pointing up in the natural reach. Roll the holder 90deg about the
tube axis (matches T1 mounting) so the seated paddle's face is lateral, aligning
with the forehand stroke. paddle_offset unchanged (blade center still ~0.337m).
Adds contact_probe.py (contact-geometry logger) and view_robot.py (empty-scene viewer).

Co-Authored-By: Claude Opus 4.8 <noreply@anthropic.com>

File: legged_lab/assets/unitree/g1_description/g1_23dof_tt_paddle.urdf (robot description, URDF)
Before this commit: robot g1_23dof_rev_1_0, 38 links, 37 joints
Joints:
- joint right_tt_paddle_holder_joint: origin xyz=0.16 0 0 rpy=0 0 0 -> xyz=0.16 0 0 rpy=1.5707963267948966 0 0

Commit message: g1_tt_v6: from-scratch retrain — stance -2.0 (>=60cm from table), 30cm arm, ankle-overrun fix, real no-ball idle
- geometry: add RobotCfg.hit_plane_x (default -1.6, G1=-2.0); parametrize all hardcoded
  -1.6/-1.65/-1.5/-1.9/-1.87 in tt_env.py (clamp/mask_invalid/mask_terminal/HOME/sentinel/
  robot_future) + rewards.py idle home; robot init pos -1.6->-2.0.
- arm 30cm: build_tt_urdf.py extension 0.16->0.123 (wrist->paddle-center 0.337->0.30),
  regenerated g1_23dof_tt_paddle.urdf (DoF preserved 23); paddle_offset 0.337->0.30.
- ankle-overrun fix: new joint_pos_target_limits (penalize commanded target exceeding soft
  limits — the missing closed loop), action_l2 (raw-action magnitude reg), joint_deviation_ankle;
  store self.processed_actions.
- real no-ball idle: no_ball_period_s 0->5 (40% cap); reward_idle_pose extended to all 23
  joints (legs/ankle ready target, ankle_roll=0 counters saturation).
- curriculum: 3-stage perf-gated (easy bootstrap -> difficulty ramp -> idle@30k), experiment g1_tt_v6.

Smoke (64env): 34 iter no NaN, new rewards active, idle gated off in stage1, fk_probe rebound OK.

Co-Authored-By: Claude Opus 4.8 <noreply@anthropic.com>

File: legged_lab/assets/unitree/g1_description/g1_23dof_tt_paddle.urdf (robot description, URDF)
Before this commit: robot g1_23dof_rev_1_0, 38 links, 37 joints
Links:
- link right_tt_extension_link: geometry collision cylinder length=0.123 radius=0.018; visual cylinder length=0.123 radius=0.018
Joints:
- joint right_tt_paddle_holder_joint: origin xyz=0.16 0 0 rpy=1.5707963267948966 0 0 -> xyz=0.123 0 0 rpy=1.5707963267948966 0 0
