Commit message: feat(a1 v3): forehand-reachable spread serve + de-park reward + 0.22kg paddle + obs norm
Fixes v2 failure (parked one pose, farmed positioning shaping, never returned to table,
critic diverged to 1e9). Root cause seen in play: hits ~70% but returns ~1.6% success.

- A (anti-park): serve spread across the MEASURED forehand-reachable envelope (FK probe:
  y in [-0.02,0.87], z in [0.50,1.52] at x=-1.42). hit_target y (0.08,0.30)->(0.0,0.55),
  z (1.08,1.32)->(0.95,1.30); widened serve_y_wide 0.08->0.27 and serve vz. One parked pose
  can no longer cover every serve -> arm must move each ball (also fixes "too slow to react").
- B: reward_future_dis_ee weight 20->4 (dense positional shaping was the park bait; it is
  already gated by mask_invalid so weight cut is the fix). Ladder contact/pass_net/landing/
  table_success now dominates positioning.
- D: action_rate_l2 -0.025->-0.01, action_l2 -0.002->-0.001 (allow faster swing).
- E: empirical_normalization=True (normalize obs) + reduced shaping magnitude -> bounds critic
  value targets (v2 had no normalization; value_loss exploded). rsl_rl has no reward/value norm.
- Paddle mass 0.15->0.22kg (real value) + inertia scaled; X1 USD regenerated via UrdfConverter.
  Verified loaded mass = 0.2200 kg.
- experiment_name a1_tt_v3; watchdog EXP default a1_tt_v3.

Verified: local smoke (32 env, 40 iters) constructs + trains, value_loss bounded (O(1-10),
not 1e9), no crash.

Co-Authored-By: Claude Opus 4.8 <noreply@anthropic.com>

File: legged_lab/assets/a1/X1_URDF_V1_1/urdf/X1_URDF_V1_1.urdf (robot description, URDF)
Before this commit: robot X1_URDF_V1_1, 31 links, 30 joints
Links:
- link Link_r_paddle: mass 0.15 -> 0.22
