Commit message: fix(a1): calibrate r1 centerline to 1.15m

File: legged_lab/assets/a1/X1_URDF_V1_3/urdf/X1_URDF_V1_3.urdf (robot description, URDF)
Before this commit: robot X1_URDF_V1_3, 31 links, 30 joints
Joints:
- joint sj: origin xyz=-0.0174775498641076 -8.52845460748708E-05 1.21100245585163 rpy=0 0 0 -> xyz=-0.0174775498641076 -8.52845460748708E-05 1.09680245585163 rpy=0 0 0
